File: kicad/aerospace_badge/aerospace_badge.kicad_pcb (KiCad board)
At the start: 2 copper layers, 134.3 x 140 mm, 20 parts, among them J1 Conn_01x02, J2 Conn_01x02, J3 Conn_02x03_Counter_Clockwise, J4 Conn_01x04, J6 Conn_01x01_Male, J7 Conn_01x01_Male, J8 Conn_01x01_Male, SW1 SW_SPDT, U1 ATtiny85-20SU

Commit message: final review with new gerbers and zip.
Other:
- board text added: "ADS-B 1090MHz"
- board text removed: "ADS-B 1090MHZ"
